File: sdwirec-hw/sdwirec.kicad_pcb (KiCad board)
At the start: 4 copper layers, 26 x 49.9 mm, 73 parts, among them IC1 USB2640-HZH-02, IC2 MC74HC1G04DTT1G, J1 USB_C_Receptacle_USB2.0, J2 usd_plug, J3 Micro_SD_Card, Q1 SMMBT4403L, Q2 SMMBT4403L, U1 M24C02-RDW, U2 SPX3819M5-L-3-3, U3 TS3A27518EPW, U4 FT200XD, Y1 24Mhz

Commit message: Update to Rev 1.4
Signed-off-by: Talha Can Havadar <talha.can.havadar@canonical.com>
Other:
- board text added: "+"
- board text added: "Rev. 1.4"
- board text removed: "Rev. 1.2"
Changed lines of the file:
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@@
   (title_block
     (title "Badgerd-SDWireC")
-    (date "2023-03-02")
-    (rev "1.2")
+    (date "2023-09-29")
+    (rev "1.4")
     (company "Badgerd Technologies B.V.")
     (comment 1 "Talha Can Havadar")
@@
     (effects (font (size 0.5 0.5) (thickness 0.1)) (justify mirror))
   )
+  (gr_text "+" (at 139.35 117.8) (layer "B.SilkS")
+    (effects (font (size 0.7 0.7) (thickness 0.1)) (justify mirror))
+  )
   (gr_text "TXD" (at 136.075 114.5) (layer "B.SilkS")
     (effects (font (size 0.5 0.5) (thickness 0.1)) (justify mirror))
   )
+  (gr_text "+" (at 139.38 119.74) (layer "B.SilkS")
+    (effects (font (size 0.7 0.7) (thickness 0.1)) (justify mirror))
+  )
   (gr_text "DEV" (at 136.095239 118.05) (layer "B.SilkS")
     (effects (font (size 0.5 0.5) (thickness 0.1)) (justify mirror))
@@
     (effects (font (size 1 1) (thickness 0.15)) (justify mirror))
   )
+  (gr_text "+" (at 139.32 116.56) (layer "B.SilkS")
+    (effects (font (size 0.7 0.7) (thickness 0.1)) (justify mirror))
+  )
+  (gr_text "+" (at 139.38 118.82) (layer "B.SilkS")
+    (effects (font (size 0.7 0.7) (thickness 0.1)) (justify mirror))
+  )
   (gr_text "PWR" (at 136 120.325) (layer "B.SilkS")
     (effects (font (size 0.5 0.5) (thickness 0.1)) (justify mirror))
   )
+  (gr_text "+" (at 139.2 114.74) (layer "B.SilkS")
+    (effects (font (size 0.7 0.7) (thickness 0.1)) (justify mirror))
+  )
   (gr_text "." (at 151.5 117.4) (layer "F.SilkS")
     (effects (font (size 1 1) (thickness 0.15)))
@@
     (effects (font (size 1 1) (thickness 0.15)))
   )
-  (gr_text "Rev. 1.2" (at 145.475 92.575) (layer "F.SilkS")
+  (gr_text "Rev. 1.4" (at 145.475 92.575) (layer "F.SilkS")
     (effects (font (size 1 1) (thickness 0.15)))
   )
